File: demonstrate.kicad_sch (KiCad schematic)
At the start: 9 parts, among them U1 ESP32-C3-WROOM-02, U2 MAX98357A, U3 AMS1117-3.3

Commit message: Added AMS1117-3V3 footprint (YIPPPEEEE)
Parts:
- added U4: ~, AMS1117-3V3:AMS1117-3V3, symbol Demo Library:Voltage_Regulator
- C1, C2, C3: footprint (none) -> Capacitor_SMD:C_0603_1608Metric
Connections:
- new net: U4.1 (GND), U4.4
